File: src/USB_JST-XH_Converter/USB_JST-XH_Converter.kicad_pcb (KiCad board)
At the start: 2 copper layers, 55.9 x 34.9 mm, 26 parts, among them SW1 SS-12D00G3

Commit message: 部品乗っけた
Parts:
- removed FET-1: IRLR6225, USB_JST-XH_Converter:TO-252AA
- removed LED1: SML-E12V8WT86, USB_JST-XH_Converter:SML-E12V8WT86
- removed PORT10, PORT11, PORT12, PORT13, PORT14, PORT6, PORT7, PORT8, PORT9: 02-JST, USB_JST-XH_Converter:B2B-XH
- added C2: GRM21BC72A105KE01, USB_JST-XH_Converter:GRM21BC72A105KE01, F.Cu at (165.6, 106.4)
- added C3: GRM1885C1H242JA01D, USB_JST-XH_Converter:GRM18, F.Cu at (161.6, 110.7)
- added C4: UWT1E221MNL1GS, USB_JST-XH_Converter:UWT1E221MNL1GS, F.Cu at (162.6, 93.4)
- added COMP1: MCP6541T-I_LT, USB_JST-XH_Converter:SC-70-5, F.Cu at (155.6, 100.4)
- added CTRL: 02-JST, USB_JST-XH_Converter:B2B-XH, F.Cu at (141.6, 118.4)
- added CTRL_I: 02-JST, USB_JST-XH_Converter:B2B-XH, F.Cu at (149.6, 118.4)
- added D1: RB751S40, USB_JST-XH_Converter:SOD-523, F.Cu at (160.6, 102.9)
- added D2: PJSD12TS, USB_JST-XH_Converter:SOD-523, F.Cu at (167.6, 106.7)
- added D3: RB751S40, USB_JST-XH_Converter:SOD-523, F.Cu at (160.6, 99.9)
- added D4: RB751S40, USB_JST-XH_Converter:SOD-523, F.Cu at (160.6, 101.4)
- added FET1: BSS138, USB_JST-XH_Converter:SOT-23, F.Cu at (157.4, 104.6)
- added IN: 03-JST, USB_JST-XH_Converter:B3B-XH, F.Cu at (146.6, 92.4)
- added JP1: PINHD-1X2, USB_JST-XH_Converter:1X02, F.Cu at (125.6, 108.4)
- added POW: SML-E12V8WT86, USB_JST-XH_Converter:SML-E12V8WT86, F.Cu at (150.1, 104.4)
- added R10: 10, USB_JST-XH_Converter:RG2012, F.Cu at (155.6, 102.9)
- added R11: 10k, USB_JST-XH_Converter:RG2012, F.Cu at (154.6, 104.9)
- added R12: 69.8k, USB_JST-XH_Converter:RG2012, F.Cu at (153.6, 108.4)
- added R13: 75k, USB_JST-XH_Converter:RG2012, F.Cu at (155.6, 108.4)
- added R14: 10k, USB_JST-XH_Converter:RG2012, F.Cu at (169.6, 112.4)
- added R4: 5.1k, USB_JST-XH_Converter:RG2012, F.Cu at (166.1, 103.4)
- added R5: 1k, USB_JST-XH_Converter:RG2012, F.Cu at (149.6, 111.9)
- added R6: 10k, USB_JST-XH_Converter:RG2012, F.Cu at (171.6, 112.4)
- added R7: 3k, USB_JST-XH_Converter:RG2012, F.Cu at (167.6, 112.4)
- added R8: 10k, USB_JST-XH_Converter:RG2012, F.Cu at (153.6, 100.0)
- added R9: 2.7k, USB_JST-XH_Converter:RG2012, F.Cu at (153.6, 97.4)
- added SW: SML-E12V8WT86, USB_JST-XH_Converter:SML-E12V8WT86, F.Cu at (150.1, 102.0)
- added SWITCH: 02-JST, USB_JST-XH_Converter:B2B-XH, F.Cu at (133.6, 118.4)
- added THRU: 03-JST, USB_JST-XH_Converter:B3B-XH, F.Cu at (135.6, 92.4)
- added TP1: GF063PB302K, USB_JST-XH_Converter:GF063PB104K, F.Cu at (154.6, 121.4)
- added TR1: 2SC3325, USB_JST-XH_Converter:2SC3325, F.Cu at (165.9, 111.9)
- added U1: TCKE805NAWSON10B_TOS-REC, USB_JST-XH_Converter:WSON10B_TOS-RIC, F.Cu at (162.1, 107.9)
- added U2: TLP293, USB_JST-XH_Converter:SO4_TOS, F.Cu at (154.6, 111.4)
- C1: value 470UF50V_NICHICON -> GRM21BC72A105KE01; footprint USB_JST-XH_Converter:470UF25V -> USB_JST-XH_Converter:GRM21BC72A105KE01
- H1, H2, H3, H4: value MOUNT-HOLE3.2 -> MOUNT-HOLE3.2(NORESIST)
- R1: value RG2012Q-100-D-T5 -> RG2012N-101-B-T5; moved to F.Cu
- R2: value RG2012 -> RG2012N-101-B-T5; moved to F.Cu
- R3: value RG2012N-101-B-T5 -> 5.1k
- USB1: value MICRO-USB -> UJC-HP-3-SMT-TR; footprint USB_JST-XH_Converter:USB_MICROB -> USB_JST-XH_Converter:UJC-HP-3-SMT-TR
- moved H2 26.5 mm to (125.1, 117.8)
- moved H1 26.5 mm to (125.1, 92.1)
- moved R1 25.2 mm to (150.6, 99.4)
- moved R2 25.1 mm to (150.6, 97.4)
- moved USB1 19.0 mm to (173.6, 103.9), turned to 90 degrees
- moved SW1 11.8 mm to (164.6, 117.3), turned to 270 degrees
- moved PORT3 11.4 mm to (142.0, 100.9)
- moved PORT2 10.9 mm to (134.0, 100.9)
- moved PORT4 10.7 mm to (134.0, 108.9)
- moved PORT1 10.6 mm to (126.0, 100.9)
- moved R3 10.4 mm to (164.1, 103.4), turned to 90 degrees
- moved PORT5 10.3 mm to (142.0, 108.9)
- moved C1 8.22 mm to (161.1, 104.9), turned to 0 degrees
- moved H3 1.11 mm to (171.9, 92.1)
- moved H4 1.10 mm to (171.9, 117.8)
Connections:
- PORT1 pad 1: SGND -> GND
- PORT2 pad 1: SGND -> GND
- PORT3 pad 1: SGND -> GND
- PORT4 pad 1: SGND -> GND
- PORT5 pad 1: SGND -> GND
- R1 pad LEFT: N$2 -> Net-(POW-PadA)
- R1 pad RIGHT: N$1 -> VCC_P
- R2 pad LEFT: N$2 -> Net-(R2-PadLEFT)
- R2 pad RIGHT: GND -> VCC
- R3 pad LEFT: N$3 -> CC1
- R3 pad RIGHT: VCC -> GND
- SW1 pad C: VCC -> SWITCH
- SW1 pad L: (no net) -> Net-(SW1-PadL)
- SW1 pad R: N$1 -> GND
Routing:
- net SGND: track 143.8 -> 0.00 mm, vias 1 -> 0
- net GND: track 22.2 -> 0.00 mm
- net N$1: track 8.57 -> 0.00 mm
- net N$2: track 5.05 -> 0.00 mm
- net N$3: track 4.33 -> 0.00 mm
- removed copper zone on B.Cu, net GND
- removed copper zone on F.Cu, net VCC
Other:
- outline, holes or cut-outs redrawn
- rule trace_min: 0.1524 -> 0.2
- board text removed: "C1"
- board text removed: "Designed by Issaimaru"
- board text removed: "FET"
- board text removed: "OFF"
- board text removed: "ON"
- board text removed: "POW"
- board text removed: "R3"
- board text removed: "USB to JST-XH"
- board text removed: "ver 1.0"
