File: src/USB_JST-XH_Converter.brd (EAGLE design)
At the start: 160 x 100 mm, 17 parts, among them P1 02-JST, P10 02-JST, P11 02-JST, P12 02-JST, P2 02-JST, P3 02-JST, P4 02-JST, P5 02-JST, P6 02-JST, P7 02-JST, P8 02-JST, P9 02-JST, SW1 SS-12D00G3

Commit message: 基板デザインの完成
Parts:
- removed P1, P10, P11, P12, P2, P3, P4, P5, P6, P7, P8, P9: 02-JST, con-jst-xh:B2B-XH
- added C1: 470UF50V_NICHICON, nichicon_470uF25V:470UF25V
- added H1, H2, H3, H4: MOUNT-HOLE3.2, holes:3,2
- added LED1: SML-E12V8WT86, SML-E12V8WT86:SML-E12V8WT86
- added PORT1, PORT10, PORT11, PORT12, PORT13, PORT14, PORT2, PORT3, PORT4, PORT5, PORT6, PORT7, PORT8, PORT9: 02-JST, con-jst-xh:B2B-XH
- added R3: RG2012N-101-B-T5, RG2012N-101-B-T5:RG2012
- moved R2 103.4 mm to (51.8, 20.6), flipped to the bottom
- moved R1 102.1 mm to (51.8, 18.4), flipped to the bottom
- moved FET-1 98.4 mm to (50.3, 23.1), flipped to the bottom
- moved SW1 81.5 mm to (40.9, 24.4)
- moved USB1 59.2 mm to (40.9, 11.8)
Connections:
- new net N$3: LED1.A, R3.LEFT
- net GND: now also C1.C-
- net SGND: now also LED1.K, PORT1.1, PORT10.1, PORT11.1, PORT12.1, PORT13.1, PORT14.1, PORT2.1, PORT3.1, PORT4.1, PORT5.1, PORT6.1, PORT7.1, PORT8.1, PORT9.1; no longer P1.1, P10.1, P11.1, P12.1, P2.1, P3.1, P4.1, P5.1, P6.1, P7.1, P8.1, P9.1
- net VCC: now also C1.C+, PORT1.2, PORT10.2, PORT11.2, PORT12.2, PORT13.2, PORT14.2, PORT2.2, PORT3.2, PORT4.2, PORT5.2, PORT6.2, PORT7.2, PORT8.2, PORT9.2, R3.RIGHT; no longer P1.2, P10.2, P11.2, P12.2, P2.2, P3.2, P4.2, P5.2, P6.2, P7.2, P8.2, P9.2
Routing:
- net SGND: track 0.00 -> 143.8 mm, vias 0 -> 1
- net GND: track 0.00 -> 22.2 mm
- net N$1: track 0.00 -> 8.57 mm
- net N$2: track 0.00 -> 5.05 mm
- net N$3: track 0.00 -> 4.33 mm
- added copper zone on layer 16, net GND
- added copper zone on layer 1, net VCC
Other:
- board size 160 x 100 mm -> 55.9 x 34.9 mm
- board text added: "C1"

Commit message: 回路図の概形大体
Parts:
- added C2, C3: GRM21BC72A105KE01, GRM21BC72A105KE01(1uF):GRM21BC72A105KE01
- added CTRL1, CTRL2, CTRL_I, SWITCH: 02-JST, con-jst-xh:B2B-XH
- added D1: (no value), diode:F126Z12
- added D2: ZZ22, diode:P2-15
- added OK1: CNF17GF, optocoupler:DIL06B
- added R10, R11, R6, R7, R8: (no value), RG2012:RG2012
- added R4, R5: 5.1k, RG2012:RG2012
- added R9: 10k, RG2012:RG2012
- added U1: TCKE805NAWSON10B_TOS-REC, TCKE805NA:WSON10B_TOS-RIC
- added U2: TC75S56F, TC75S56F:SOT-25___(SMV)_TOS
- C1: value 470UF50V_NICHICON -> GRM21BC72A105KE01; device nichicon_470uF25V:470UF25V -> GRM21BC72A105KE01(1uF):GRM21BC72A105KE01
- H1, H2, H3, H4: value MOUNT-HOLE3.2 -> MOUNT-HOLE3.2(NORESIST); device holes:3,2 -> MOUNT-HOLE3.2(NORESIST):3,2
- R2: value RG2012 -> 10k
- USB1: value MICRO-USB -> UJC-HP-3-SMT-TR; device USB-MICROB:USB_MICROB -> UJC-HP-3-SMT-TR:UJC-HP-3-SMT-TR
- moved C1 99.0 mm to (-37.0, -26.0), turned to 0 degrees
- moved USB1 46.3 mm to (-3.00, -3.00)
- moved H2 26.5 mm to (4.80, 12.6)
- moved H1 26.5 mm to (4.60, 38.3)
- moved H3 1.11 mm to (51.3, 38.3)
- moved H4 1.10 mm to (51.3, 12.6)
Connections:
- new net N$10: OK1.2, R9.LEFT
- new net N$11: R10.RIGHT, R11.RIGHT, U2.3
- new net N$4: R4.LEFT, USB1.A5
- new net N$5: R5.LEFT, USB1.B5
- new net N$6: R6.RIGHT, U1.ILIM
- new net N$7: C3.P$1, U1.DVDT
- new net N$8: CTRL_I.2, OK1.1
- new net N$9: CTRL_I.1, R9.RIGHT
- new net SWITCH: CTRL1.1, CTRL2.1, OK1.5, R7.LEFT, R8.RIGHT, SWITCH.1, U1.EN/UVLO
- new net VCC_P: C2.P$1, D2.C, R10.LEFT, R7.RIGHT, U1.VIN1, U1.VIN2, U1.VIN3, USB1.A9, USB1.B9
- net GND: now also C1.P$2, C2.P$2, C3.P$2, D1.A, D2.A, H1.P$1, H2.P$1, H3.P$1, H4.P$1, OK1.4, R11.LEFT, R4.RIGHT, R5.RIGHT, R6.LEFT, R8.LEFT, SWITCH.2, U1.GND1, U1.GND2, U1.GND3, U1.GND4, U1.GND5, USB1.A12, USB1.B12, USB1.SHIELD1, USB1.SHIELD2, USB1.SHIELD3, USB1.SHIELD4; no longer C1.C-, USB1.GND1, USB1.GND2, USB1.USB-
- net VCC: now also C1.P$1, D1.C, U1.VOUT1, U1.VOUT2, U1.VOUT3; no longer C1.C+, USB1.USB+
Routing:
- net GND: track 22.2 -> 14.3 mm
- added copper zone on layer 1, net GND
- removed copper zone on layer 1, net VCC
Other:
- outline, holes or cut-outs redrawn

Commit message: 回路図仮完成
Parts:
- removed FET-1: IRLR6225, OKUDA_libraries:TO-252AA
- removed OK1: CNF17GF, optocoupler:DIL06B
- removed PORT10, PORT11, PORT12, PORT13, PORT14, PORT9: 02-JST, con-jst-xh:B2B-XH
- removed R2, R9: 10k, RG2012:RG2012
- added C4: UWT1E221MNL1GS, UWT1E221MNL1GS:UWT1E221MNL1GS
- added COMP1: MCP6541T-I/LT, MCP6541T-I:SC-70-5
- added D3, D4: RB751S40, RB751S40:SOD-523
- added FET1: BSS138, BSS138:SOT-23
- added IN, THRU: (no value), con-jst-xh:B3B-XH
- added JP1: (no value), pinhead:1X02
- added POW: SML-E12V8WT86, SML-E12V8WT86:SML-E12V8WT86
- added R12: 10, RG2012:RG2012
- added R13, R16: 10k, RG2012:RG2012
- added R14: 69.8k, RG2012:RG2012
- added R15: 75k, RG2012:RG2012
- added TP1: GF063PB302K, GF063P B104K:GF063PB104K
- added TR1: 2SC3325, 2SC3325:2SC3325
- C3: value GRM21BC72A105KE01 -> GRM1885C1H242JA01D; device GRM21BC72A105KE01(1uF):GRM21BC72A105KE01 -> GRM1885C1H242JA01D:GRM18
- D1: value (none) -> RB751S40; device diode:F126Z12 -> RB751S40:SOD-523
- D2: value ZZ22 -> PJSD12TS; device diode:P2-15 -> PJSD12TS:SOD-523
- R1: value RG2012Q-100-D-T5 -> RG2012N-101-B-T5; device RG2012Q-100-D-T5:RG2012 -> RG2012N-101-B-T5:RG2012
- R10, R7: value (none) -> 10k
- R11: value (none) -> 2.7k
- R6: value (none) -> 1k
- R8: value (none) -> 3k
- U2: value TC75S56F -> TLP293; device TC75S56F:SOT-25___(SMV)_TOS -> TLP293:SO4_TOS
- USB1: device UJC-HP-3-SMT-TR:UJC-HP-3-SMT-TR -> UJC-HP-3-SMT-TRv2:UJC-HP-3-SMT-TR
- moved R11 158.6 mm to (28.0, 53.0)
- moved R10 158.1 mm to (28.0, 56.0)
- moved C1 127.3 mm to (43.0, 73.0)
- moved C2 127.3 mm to (43.0, 70.0)
- moved CTRL2 127.3 mm to (23.0, 51.0)
- moved R7 127.3 mm to (42.0, 53.0)
- moved R8 127.3 mm to (42.0, 50.0)
- moved U2 124.5 mm to (42.0, 30.0)
- moved D2 110.1 mm to (11.0, 67.0)
- moved C3 105.6 mm to (47.0, 21.0)
- moved CTRL1 104.7 mm to (25.0, 86.0)
- moved CTRL_I 104.7 mm to (15.0, 86.0)
- moved R4 104.7 mm to (43.0, 85.0)
- moved R5 104.7 mm to (43.0, 82.0)
- moved SWITCH 104.7 mm to (35.0, 86.0)
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- renumbered LED1 to SW
Connections:
- removed net N$11: R10.RIGHT, R11.RIGHT, U2.3
- removed net SGND: FET-1.D, PORT1.1, PORT10.1, PORT11.1, PORT12.1, PORT13.1, PORT14.1, PORT2.1, PORT3.1, PORT4.1, PORT5.1, PORT6.1, PORT7.1, PORT8.1, PORT9.1, SW.K
- new net CC: COMP1.IN+, D3.C, D4.C, IN.2, THRU.2
- new net CC1: D3.A, R4.LEFT, USB1.A5
- new net CC2: D4.A, R5.LEFT, USB1.B5
- new net ILIM: R14.LEFT, R15.LEFT, U1.ILIM
- new net N$12: COMP1.OUT, R12.RIGHT
- new net N$15: FET1.D, R14.RIGHT
- net GND: now also C3.R, C4.C, COMP1.VSS, FET1.S, IN.1, JP1.2, PORT1.1, PORT2.1, PORT3.1, PORT4.1, PORT5.1, PORT6.1, PORT7.1, PORT8.1, POW.K, R11.RIGHT, R13.RIGHT, R15.RIGHT, SW.K, SW1.R, THRU.1, TR1.E, U2.3; no longer C3.P$2, FET-1.S, OK1.4, R11.LEFT, R2.RIGHT, R6.LEFT
- net N$1: now also POW.A, R1.LEFT; no longer R1.RIGHT, SW1.R
- net N$10: now also R6.LEFT, U2.2; no longer OK1.2, R9.LEFT
- net N$2: now also R8.RIGHT, TP1.LEFT, TR1.C, U1.EN/UVLO; no longer FET-1.G, R1.LEFT, R2.LEFT
- net N$4: now also COMP1.IN-, R10.LEFT, R11.LEFT; no longer R4.LEFT, USB1.A5
- net N$5: now also FET1.G, R12.LEFT, R13.LEFT; no longer R5.LEFT, USB1.B5
- net N$6: now also R7.LEFT, TP1.CENTER, TP1.RIGHT; no longer R6.RIGHT, U1.ILIM
- net N$7: now also C3.L; no longer C3.P$1
- net N$8: now also U2.1; no longer OK1.1
- net N$9: now also R6.RIGHT; no longer R9.RIGHT
- net SWITCH: now also JP1.1, R16.LEFT, SW1.C, TR1.B, U2.4; no longer OK1.5, R7.LEFT, R8.RIGHT, U1.EN/UVLO
- net VCC: now also C4.A; no longer PORT10.2, PORT11.2, PORT12.2, PORT13.2, PORT14.2, PORT9.2, SW1.C
- net VCC_P: now also COMP1.VDD, IN.3, R1.RIGHT, R10.RIGHT, R16.RIGHT, THRU.3; no longer R10.LEFT
Routing:
- net SGND: track 143.8 -> 0.00 mm, vias 1 -> 0
- net GND: track 14.3 -> 0.00 mm
- net N$1: track 8.57 -> 0.00 mm
- net N$2: track 5.05 -> 0.00 mm
- net N$3: track 4.33 -> 0.00 mm
- removed copper zone on layer 1, net GND
- removed copper zone on layer 16, net GND

Commit message: 部品乗っけた
Parts:
- removed CTRL1, CTRL2, PORT6, PORT7, PORT8: 02-JST, con-jst-xh:B2B-XH
- removed R15: 75k, RG2012:RG2012
- removed R16: 10k, RG2012:RG2012
- added CTRL: 02-JST, con-jst-xh:B2B-XH
- added R2: RG2012N-101-B-T5, RG2012N-101-B-T5:RG2012
- added R9: 2.7k, RG2012:RG2012
- R10: value 10k -> 10
- R11: value 2.7k -> 10k
- R12: value 10 -> 69.8k
- R13: value 10k -> 75k
- R14: value 69.8k -> 10k
- R3: value RG2012N-101-B-T5 -> 5.1k; device RG2012N-101-B-T5:RG2012 -> RG2012:RG2012
- R5: value 5.1k -> 1k
- R6: value 1k -> 10k
- R7: value 10k -> 3k
- R8: value 3k -> 10k
- moved C4 89.3 mm to (42.0, 37.0)
- moved U1 87.3 mm to (41.5, 22.5), turned to 180 degrees
- moved SWITCH 77.2 mm to (13.0, 12.0)
- moved CTRL_I 75.3 mm to (29.0, 12.0)
- moved TP1 65.9 mm to (34.0, 9.00)
- moved R6 65.2 mm to (51.0, 18.0), turned to 90 degrees
- moved R5 65.0 mm to (29.0, 18.5), turned to 180 degrees
- moved POW 63.0 mm to (29.5, 26.0), turned to 90 degrees
- moved R4 58.1 mm to (45.5, 27.0), turned to 90 degrees
- moved R1 57.2 mm to (30.0, 31.0), turned to 180 degrees
- moved D2 56.3 mm to (47.0, 23.7), turned to 90 degrees
- moved FET1 55.6 mm to (36.8, 25.8), turned to 180 degrees
- moved C1 47.6 mm to (40.5, 25.5)
- moved D1 47.4 mm to (40.0, 27.5)
- moved C2 46.0 mm to (45.0, 24.0), turned to 90 degrees
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Connections:
- net CC1: now also R3.LEFT; no longer R4.LEFT
- net CC2: now also R4.LEFT; no longer R5.LEFT
- net GND: now also R3.RIGHT, R7.LEFT, R9.RIGHT; no longer PORT6.1, PORT7.1, PORT8.1, R15.RIGHT, R5.RIGHT, R8.LEFT
- net ILIM: now also R12.LEFT, R13.LEFT; no longer R14.LEFT, R15.LEFT
- net N$10: now also R5.LEFT; no longer R6.LEFT
- net N$12: now also R10.RIGHT; no longer R12.RIGHT
- net N$15: now also R12.RIGHT; no longer R14.RIGHT
- net N$2: now also R7.RIGHT; no longer R8.RIGHT
- net N$3: now also R2.LEFT; no longer R3.LEFT
- net N$4: now also R8.LEFT, R9.LEFT; no longer R10.LEFT, R11.LEFT
- net N$5: now also R10.LEFT, R11.LEFT; no longer R12.LEFT, R13.LEFT
- net N$6: now also R6.LEFT; no longer R7.LEFT
- net N$9: now also R5.RIGHT; no longer R6.RIGHT
- net SWITCH: now also CTRL.1, R14.LEFT; no longer CTRL1.1, CTRL2.1, R16.LEFT
- net VCC: now also R2.RIGHT; no longer PORT6.2, PORT7.2, PORT8.2, R3.RIGHT
- net VCC_P: now also R14.RIGHT, R6.RIGHT, R8.RIGHT; no longer R10.RIGHT, R16.RIGHT, R7.RIGHT
Other:
- board text removed: "C1"

Commit message: 配線完了
Parts:
- moved THRU 26.0 mm to (41.0, 38.0)
- moved C4 25.1 mm to (17.0, 39.0)
- moved D4 3.50 mm to (40.0, 32.5)
- moved IN 3.00 mm to (29.0, 38.0)
- moved R13 3.00 mm to (38.0, 22.0), turned to 180 degrees
- moved R1 2.69 mm to (27.5, 32.0), turned to 0 degrees
- moved R2 2.69 mm to (27.5, 34.0), turned to 0 degrees
- moved POW 2.51 mm to (27.2, 27.0), turned to 270 degrees
- moved SW 2.38 mm to (27.2, 29.0), turned to 270 degrees
- moved C1 2.00 mm to (40.5, 27.5)
- moved COMP1 2.00 mm to (35.0, 32.0)
- moved D1 2.00 mm to (40.0, 29.5)
- moved FET1 2.00 mm to (36.8, 27.8)
- moved R10 2.00 mm to (35.0, 29.5)
- moved R11 2.00 mm to (34.0, 27.5)
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Routing:
- net SWITCH: track 0.00 -> 74.9 mm
- net GND: track 0.00 -> 38.5 mm, vias 0 -> 37
- net VCC_P: track 0.00 -> 28.3 mm, vias 0 -> 2
- net CC: track 0.00 -> 20.5 mm
- net VCC: track 0.00 -> 19.9 mm
- net N$2: track 0.00 -> 19.7 mm
- net N$6: track 0.00 -> 17.0 mm
- net CC2: track 0.00 -> 13.4 mm, vias 0 -> 2
- net N$9: track 0.00 -> 12.2 mm
- net CC1: track 0.00 -> 12.0 mm, vias 0 -> 2
- net N$15: track 0.00 -> 11.4 mm, vias 0 -> 2
- net N$8: track 0.00 -> 10.5 mm
- net ILIM: track 0.00 -> 9.34 mm
- net N$3: track 0.00 -> 7.10 mm
- net N$1: track 0.00 -> 6.43 mm
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- added copper zone on layer 1, net GND
- added copper zone on layer 16, net GND
- added copper zone on layer 1, net VCC
- added copper zone on layer 1, net VCC_P
Other:
- board size 55.9 x 34.9 mm -> 55.9 x 35.9 mm
