File: src/USB_JST-XH_Converter.sch (EAGLE design)
At the start: 17 parts, among them P1 02-JST, P10 02-JST, P11 02-JST, P12 02-JST, P2 02-JST, P3 02-JST, P4 02-JST, P5 02-JST, P6 02-JST, P7 02-JST, P8 02-JST, P9 02-JST, SW1 SS-12D00G3

Commit message: 基板デザインの完成
Parts:
- added C1: 470UF50V_NICHICON, nichicon_470uF25V:470UF50V_NICHICON
- added H1, H2, H3, H4: MOUNT-HOLE3.2, holes:MOUNT-HOLE3.2
- added LED1: SML-E12V8WT86, SML-E12V8WT86:SML-E12V8WT86
- added PORT13, PORT14: 02-JST, con-jst-xh:02-JST
- added R3: RG2012N-101-B-T5, RG2012N-101-B-T5:RG2012N-101-B-T5
- renumbered P1 to PORT1, P10 to PORT10, P11 to PORT11, P12 to PORT12, P2 to PORT2, P3 to PORT3, P4 to PORT4, P5 to PORT5, P6 to PORT6, P7 to PORT7, P8 to PORT8, P9 to PORT9
Connections:
- new net N$3: LED1.A, R3.P$1
- net GND: now also C1.CATHODE
- net SGND: now also LED1.C, PORT13.1, PORT14.1
- net VCC: now also C1.ANODE, PORT13.2, PORT14.2, R3.P$2
Other:
- note added: "LED"

Commit message: 回路図の概形大体
Parts:
- added C2, C3: GRM21BC72A105KE01, GRM21BC72A105KE01(1uF):GRM21BC72A105KE01
- added CTRL1, CTRL2, CTRL_I, SWITCH: 02-JST, con-jst-xh:02-JST
- added D1: (no value), diode:SCHOTTKY-DIODEF126Z12
- added D2: ZZ22, diode:ZZ22
- added OK1: CNF17GF, optocoupler:CNF17GF
- added R10, R11, R6, R7, R8: (no value), RG2012:RG2012
- added R4, R5: 5.1k, RG2012:RG2012
- added R9: 10k, RG2012:RG2012
- added U1: TCKE805NAWSON10B_TOS-REC, TCKE805NA:TCKE805NAWSON10B_TOS-REC
- added U2: TC75S56F, TC75S56F:TC75S56F
- C1: value 470UF50V_NICHICON -> GRM21BC72A105KE01; device nichicon_470uF25V:470UF50V_NICHICON -> GRM21BC72A105KE01(1uF):GRM21BC72A105KE01
- H1, H2, H3, H4: value MOUNT-HOLE3.2 -> MOUNT-HOLE3.2(NORESIST); device holes:MOUNT-HOLE3.2 -> MOUNT-HOLE3.2(NORESIST):MOUNT-HOLE3.2(NORESIST)
- R2: value RG2012 -> 10k
- USB1: value MICRO-USB -> UJC-HP-3-SMT-TR; device USB-MICROB:MICRO-USB -> UJC-HP-3-SMT-TR:UJC-HP-3-SMT-TR
Connections:
- new net N$10: OK1.C, R9.LEFT
- new net N$11: R10.RIGHT, R11.RIGHT, U2.3
- new net N$4: R4.LEFT, USB1.CC1
- new net N$5: R5.LEFT, USB1.CC2
- new net N$6: R6.RIGHT, U1.ILIM
- new net N$7: C3.P$1, U1.DV/DT
- new net N$8: CTRL_I.2, OK1.A
- new net N$9: CTRL_I.1, R9.RIGHT
- new net SWITCH: CTRL1.1, CTRL2.1, OK1.COL, R7.LEFT, R8.RIGHT, SWITCH.1, U1.EN/UVLO
- new net VCC_P: C2.P$1, D2.2, R10.LEFT, R7.RIGHT, U1.VIN, U1.VIN_2, U1.VIN_3, USB1.V-BUS
- net GND: now also C1.P$2, C2.P$2, C3.P$2, D1.A, D2.1, H1.P$1, H2.P$1, H3.P$1, H4.P$1, OK1.EMIT, R11.LEFT, R4.RIGHT, R5.RIGHT, R6.LEFT, R8.LEFT, SWITCH.2, U1.GND, USB1.GND, USB1.SHIELD; no longer C1.CATHODE, USB1.USB-
- net VCC: now also C1.P$1, D1.C, U1.VOUT, U1.VOUT_2, U1.VOUT_3; no longer C1.ANODE, USB1.USB+

Commit message: 回路図仮完成
Parts:
- removed FET-1: IRLR6225, OKUDA_libraries:IRLR6225
- removed LED1: SML-E12V8WT86, SML-E12V8WT86:SML-E12V8WT86
- removed OK1: CNF17GF, optocoupler:CNF17GF
- removed PORT10, PORT11, PORT12, PORT13, PORT14, PORT9: 02-JST, con-jst-xh:02-JST
- removed R2, R9: 10k, RG2012:RG2012
- added C4: UWT1E221MNL1GS, UWT1E221MNL1GS:UWT1E221MNL1GS
- added COMP1: MCP6541T-I/LT, MCP6541T-I:MCP6541T-I/LT
- added D3, D4: RB751S40, RB751S40:RB751S40
- added FET1: BSS138, BSS138:BSS138
- added IN, THRU: (no value), con-jst-xh:03-JST
- added JP1: (no value), pinhead:PINHD-1X2
- added POW, SW: SML-E12V8WT86, SML-E12V8WT86:SML-E12V8WT86
- added R12: 10, RG2012:RG2012
- added R13, R16: 10k, RG2012:RG2012
- added R14: 69.8k, RG2012:RG2012
- added R15: 75k, RG2012:RG2012
- added TP1: GF063PB302K, GF063P B104K:GF063PB302K
- added TR1: 2SC3325, 2SC3325:2SC3325
- C3: value GRM21BC72A105KE01 -> GRM1885C1H242JA01D; device GRM21BC72A105KE01(1uF):GRM21BC72A105KE01 -> GRM1885C1H242JA01D:GRM1885C1H242JA01D
- D1: value (none) -> RB751S40; device diode:SCHOTTKY-DIODEF126Z12 -> RB751S40:RB751S40
- D2: value ZZ22 -> PJSD12TS; device diode:ZZ22 -> PJSD12TS:PJSD12TS
- R1: value RG2012Q-100-D-T5 -> RG2012N-101-B-T5; device RG2012Q-100-D-T5:RG2012Q-100-D-T5 -> RG2012N-101-B-T5:RG2012N-101-B-T5
- R10, R7: value (none) -> 10k
- R11: value (none) -> 2.7k
- R6: value (none) -> 1k
- R8: value (none) -> 3k
- U2: value TC75S56F -> TLP293; device TC75S56F:TC75S56F -> TLP293:TLP293
- USB1: device UJC-HP-3-SMT-TR:UJC-HP-3-SMT-TR -> UJC-HP-3-SMT-TRv2:UJC-HP-3-SMT-TR
Connections:
- removed net N$11: R10.RIGHT, R11.RIGHT, U2.3
- removed net SGND: FET-1.D, LED1.C, PORT1.1, PORT10.1, PORT11.1, PORT12.1, PORT13.1, PORT14.1, PORT2.1, PORT3.1, PORT4.1, PORT5.1, PORT6.1, PORT7.1, PORT8.1, PORT9.1
- new net CC: COMP1.IN+, D3.C, D4.C, IN.2, THRU.2
- new net CC1: D3.A, R4.LEFT, USB1.CC1
- new net CC2: D4.A, R5.LEFT, USB1.CC2
- new net ILIM: R14.LEFT, R15.LEFT, U1.ILIM
- new net N$12: COMP1.OUT, R12.RIGHT
- new net N$15: FET1.D, R14.RIGHT
- net GND: now also C3.2, C4.CATHODE, COMP1.VSS, D2.A, FET1.S, IN.1, JP1.2, PORT1.1, PORT2.1, PORT3.1, PORT4.1, PORT5.1, PORT6.1, PORT7.1, PORT8.1, POW.C, R11.RIGHT, R13.RIGHT, R15.RIGHT, SW.C, SW1.R, THRU.1, TR1.E, U2.3; no longer C3.P$2, D2.1, FET-1.S, OK1.EMIT, R11.LEFT, R2.RIGHT, R6.LEFT
- net N$1: now also POW.A, R1.P$1; no longer R1.P$2, SW1.R
- net N$10: now also R6.LEFT, U2.2; no longer OK1.C, R9.LEFT
- net N$2: now also R8.RIGHT, TP1.LEFT, TR1.C, U1.EN/UVLO; no longer FET-1.G, R1.P$1, R2.LEFT
- net N$3: now also SW.A; no longer LED1.A
- net N$4: now also COMP1.IN-, R10.LEFT, R11.LEFT; no longer R4.LEFT, USB1.CC1
- net N$5: now also FET1.G, R12.LEFT, R13.LEFT; no longer R5.LEFT, USB1.CC2
- net N$6: now also R7.LEFT, TP1.RIGHT; no longer R6.RIGHT, U1.ILIM
- net N$7: now also C3.1; no longer C3.P$1
- net N$8: now also U2.1; no longer OK1.A
- net N$9: now also R6.RIGHT; no longer R9.RIGHT
- net SWITCH: now also JP1.1, R16.LEFT, SW1.C, TR1.B, U2.4; no longer OK1.COL, R7.LEFT, R8.RIGHT, U1.EN/UVLO
- net VCC: now also C4.ANODE; no longer PORT10.2, PORT11.2, PORT12.2, PORT13.2, PORT14.2, PORT9.2, SW1.C
- net VCC_P: now also COMP1.VDD, D2.C, IN.3, R1.P$2, R10.RIGHT, R16.RIGHT, THRU.3; no longer D2.2, R10.LEFT
Other:
- note added: "CTRL"
- note added: "Current Supply Capability Discrimination Circuit"
- note added: "POW"
- note added: "POW_LED"
- note added: "SWITCH_LED"
- note added: "eFuse"
- note added: "完"
- note removed: "LED"
- moved on the sheet: C1, C2, CTRL1, CTRL2, CTRL_I, D1, PORT1, PORT2, PORT3, PORT4, PORT5, PORT6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

Commit message: 部品乗っけた
Parts:
- removed CTRL1, CTRL2, PORT6, PORT7, PORT8: 02-JST, con-jst-xh:02-JST
- removed R15: 75k, RG2012:RG2012
- removed R16: 10k, RG2012:RG2012
- added CTRL: 02-JST, con-jst-xh:02-JST
- added R2: RG2012N-101-B-T5, RG2012N-101-B-T5:RG2012N-101-B-T5
- added R9: 2.7k, RG2012:RG2012
- R10: value 10k -> 10
- R11: value 2.7k -> 10k
- R12: value 10 -> 69.8k
- R13: value 10k -> 75k
- R14: value 69.8k -> 10k
- R3: value RG2012N-101-B-T5 -> 5.1k; device RG2012N-101-B-T5:RG2012N-101-B-T5 -> RG2012:RG2012
- R5: value 5.1k -> 1k
- R6: value 1k -> 10k
- R7: value 10k -> 3k
- R8: value 3k -> 10k
Connections:
- net CC1: now also R3.LEFT; no longer R4.LEFT
- net CC2: now also R4.LEFT; no longer R5.LEFT
- net GND: now also R3.RIGHT, R7.LEFT, R9.RIGHT; no longer PORT6.1, PORT7.1, PORT8.1, R15.RIGHT, R5.RIGHT, R8.LEFT
- net ILIM: now also R12.LEFT, R13.LEFT; no longer R14.LEFT, R15.LEFT
- net N$10: now also R5.LEFT; no longer R6.LEFT
- net N$12: now also R10.RIGHT; no longer R12.RIGHT
- net N$15: now also R12.RIGHT; no longer R14.RIGHT
- net N$2: now also R7.RIGHT; no longer R8.RIGHT
- net N$3: now also R2.P$1; no longer R3.P$1
- net N$4: now also R8.LEFT, R9.LEFT; no longer R10.LEFT, R11.LEFT
- net N$5: now also R10.LEFT, R11.LEFT; no longer R12.LEFT, R13.LEFT
- net N$6: now also R6.LEFT; no longer R7.LEFT
- net N$9: now also R5.RIGHT; no longer R6.RIGHT
- net SWITCH: now also CTRL.1, R14.LEFT; no longer CTRL1.1, CTRL2.1, R16.LEFT
- net VCC: now also R2.P$2; no longer PORT6.2, PORT7.2, PORT8.2, R3.P$2
- net VCC_P: now also R14.RIGHT, R6.RIGHT, R8.RIGHT; no longer R10.RIGHT, R16.RIGHT, R7.RIGHT
Other:
- moved on the sheet: R10, R11, R12, R13, R4, R5, R7, SWITCH

Commit message: 配線完了
Other:
- moved on the sheet: PORT1, PORT2, PORT3, PORT4, PORT5
Changed lines of the file:
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@@
 <sheet>
 <plain>
-<wire x1="8.89" y1="74.93" x2="8.89" y2="35.56" width="0.1524" layer="97"/>
-<wire x1="8.89" y1="35.56" x2="105.41" y2="35.56" width="0.1524" layer="97"/>
-<wire x1="105.41" y1="35.56" x2="105.41" y2="74.93" width="0.1524" layer="97"/>
-<wire x1="105.41" y1="74.93" x2="8.89" y2="74.93" width="0.1524" layer="97"/>
+<wire x1="24.13" y1="74.93" x2="24.13" y2="35.56" width="0.1524" layer="97"/>
+<wire x1="24.13" y1="35.56" x2="95.25" y2="35.56" width="0.1524" layer="97"/>
+<wire x1="95.25" y1="35.56" x2="95.25" y2="74.93" width="0.1524" layer="97"/>
+<wire x1="95.25" y1="74.93" x2="24.13" y2="74.93" width="0.1524" layer="97"/>
 <wire x1="118.11" y1="55.88" x2="118.11" y2="27.94" width="0.1524" layer="97"/>
 <wire x1="118.11" y1="27.94" x2="170.18" y2="27.94" width="0.1524" layer="97"/>
@@
 <wire x1="170.18" y1="55.88" x2="118.11" y2="55.88" width="0.1524" layer="97"/>
 <text x="139.7" y="25.4" size="1.778" layer="97">Switch</text>
-<text x="53.34" y="33.02" size="1.778" layer="97">Port</text>
+<text x="55.88" y="33.02" size="1.778" layer="97">Port</text>
 <text x="30.734" y="86.614" size="1.778" layer="97" rot="MR0">USB</text>
 <wire x1="56.896" y1="97.79" x2="56.896" y2="83.82" width="0.1524" layer="97"/>
@@
 <attribute name="SHEET" x="154.305" y="5.08" size="2.54" layer="94"/>
 </instance>
-<instance part="PORT1" gate="G$1" x="16.51" y="66.04" smashed="yes">
-<attribute name="VALUE" x="15.24" y="58.42" size="1.778" layer="96"/>
-<attribute name="NAME" x="15.24" y="69.342" size="1.778" layer="95"/>
-</instance>
-<instance part="PORT2" gate="G$1" x="36.83" y="66.04" smashed="yes">
-<attribute name="VALUE" x="35.56" y="58.42" size="1.778" layer="96"/>
-<attribute name="NAME" x="35.56" y="69.342" size="1.778" layer="95"/>
-</instance>
-<instance part="PORT3" gate="G$1" x="58.42" y="66.04" smashed="yes">
-<attribute name="VALUE" x="57.15" y="58.42" size="1.778" layer="96"/>
-<attribute name="NAME" x="57.15" y="69.342" size="1.778" layer="95"/>
-</instance>
-<instance part="PORT4" gate="G$1" x="78.74" y="66.04" smashed="yes">
-<attribute name="VALUE" x="77.47" y="58.42" size="1.778" layer="96"/>
-<attribute name="NAME" x="77.47" y="69.342" size="1.778" layer="95"/>
-</instance>
-<instance part="PORT5" gate="G$1" x="16.51" y="48.26" smashed="yes">
-<attribute name="VALUE" x="15.24" y="40.64" size="1.778" layer="96"/>
-<attribute name="NAME" x="15.24" y="51.562" size="1.778" layer="95"/>
+<instance part="PORT1" gate="G$1" x="31.75" y="66.04" smashed="yes">
+<attribute name="VALUE" x="30.48" y="58.42" size="1.778" layer="96"/>
+<attribute name="NAME" x="30.48" y="69.342" size="1.778" layer="95"/>
+</instance>
+<instance part="PORT2" gate="G$1" x="52.07" y="66.04" smashed="yes">
+<attribute name="VALUE" x="50.8" y="58.42" size="1.778" layer="96"/>
+<attribute name="NAME" x="50.8" y="69.342" size="1.778" layer="95"/>
+</instance>
+<instance part="PORT3" gate="G$1" x="73.66" y="66.04" smashed="yes">
+<attribute name="VALUE" x="72.39" y="58.42" size="1.778" layer="96"/>
+<attribute name="NAME" x="72.39" y="69.342" size="1.778" layer="95"/>
+</instance>
+<instance part="PORT4" gate="G$1" x="31.75" y="48.514" smashed="yes">
+<attribute name="VALUE" x="30.48" y="40.894" size="1.778" layer="96"/>
+<attribute name="NAME" x="30.48" y="51.816" size="1.778" layer="95"/>
+</instance>
+<instance part="PORT5" gate="G$1" x="52.07" y="48.26" smashed="yes">
+<attribute name="VALUE" x="50.8" y="40.64" size="1.778" layer="96"/>
+<attribute name="NAME" x="50.8" y="51.562" size="1.778" layer="95"/>
 </instance>
 <instance part="SW1" gate="G$1" x="143.51" y="43.18" smashed="yes" rot="R270">
@@
 <segment>
 <pinref part="PORT1" gate="G$1" pin="2"/>
-<wire x1="24.13" y1="66.04" x2="29.21" y2="66.04" width="0.1524" layer="91"/>
-<label x="25.4" y="66.04" size="1.778" layer="95"/>
+<wire x1="39.37" y1="66.04" x2="44.45" y2="66.04" width="0.1524" layer="91"/>
+<label x="40.64" y="66.04" size="1.778" layer="95"/>
 </segment>
 <segment>
 <pinref part="PORT2" gate="G$1" pin="2"/>
-<wire x1="44.45" y1="66.04" x2="50.8" y2="66.04" width="0.1524" layer="91"/>
-<label x="46.99" y="66.04" size="1.778" layer="95"/>
+<wire x1="59.69" y1="66.04" x2="66.04" y2="66.04" width="0.1524" layer="91"/>
+<label x="62.23" y="66.04" size="1.778" layer="95"/>
 </segment>
 <segment>
 <pinref part="PORT3" gate="G$1" pin="2"/>
-<wire x1="66.04" y1="66.04" x2="72.39" y2="66.04" width="0.1524" layer="91"/>
-<label x="68.58" y="66.04" size="1.778" layer="95"/>
+<wire x1="81.28" y1="66.04" x2="87.63" y2="66.04" width="0.1524" layer="91"/>
+<label x="83.82" y="66.04" size="1.778" layer="95"/>
 </segment>
 <segment>
 <pinref part="PORT4" gate="G$1" pin="2"/>
-<wire x1="86.36" y1="66.04" x2="92.71" y2="66.04" width="0.1524" layer="91"/>
-<label x="88.9" y="66.04" size="1.778" layer="95"/>
+<wire x1="39.37" y1="48.514" x2="45.72" y2="48.514" width="0.1524" layer="91"/>
+<label x="41.91" y="48.514" size="1.778" layer="95"/>
 </segment>
 <segment>
 <pinref part="PORT5" gate="G$1" pin="2"/>
-<wire x1="24.13" y1="48.26" x2="29.21" y2="48.26" width="0.1524" layer="91"/>
-<label x="25.4" y="48.26" size="1.778" layer="95"/>
+<wire x1="59.69" y1="48.26" x2="64.77" y2="48.26" width="0.1524" layer="91"/>
+<label x="60.96" y="48.26" size="1.778" layer="95"/>
 </segment>
 <segment>
@@
 <segment>
 <pinref part="PORT5" gate="G$1" pin="1"/>
-<wire x1="24.13" y1="45.72" x2="29.21" y2="45.72" width="0.1524" layer="91"/>
-<label x="25.4" y="45.72" size="1.778" layer="95"/>
+<wire x1="59.69" y1="45.72" x2="64.77" y2="45.72" width="0.1524" layer="91"/>
+<label x="60.96" y="45.72" size="1.778" layer="95"/>
 </segment>
 <segment>
 <pinref part="PORT1" gate="G$1" pin="1"/>
-<wire x1="24.13" y1="63.5" x2="29.21" y2="63.5" width="0.1524" layer="91"/>
-<label x="25.4" y="63.5" size="1.778" layer="95"/>
+<wire x1="39.37" y1="63.5" x2="44.45" y2="63.5" width="0.1524" layer="91"/>
+<label x="40.64" y="63.5" size="1.778" layer="95"/>
 </segment>
 <segment>
 <pinref part="PORT2" gate="G$1" pin="1"/>
-<wire x1="44.45" y1="63.5" x2="50.8" y2="63.5" width="0.1524" layer="91"/>
-<label x="46.99" y="63.5" size="1.778" layer="95"/>
+<wire x1="59.69" y1="63.5" x2="66.04" y2="63.5" width="0.1524" layer="91"/>
+<label x="62.23" y="63.5" size="1.778" layer="95"/>
 </segment>
 <segment>
 <pinref part="PORT3" gate="G$1" pin="1"/>
-<wire x1="66.04" y1="63.5" x2="72.39" y2="63.5" width="0.1524" layer="91"/>
-<label x="68.58" y="63.5" size="1.778" layer="95"/>
+<wire x1="81.28" y1="63.5" x2="87.63" y2="63.5" width="0.1524" layer="91"/>
+<label x="83.82" y="63.5" size="1.778" layer="95"/>
 </segment>
 <segment>
 <pinref part="PORT4" gate="G$1" pin="1"/>
-<wire x1="86.36" y1="63.5" x2="92.71" y2="63.5" width="0.1524" layer="91"/>
-<label x="88.9" y="63.5" size="1.778" layer="95"/>
-</segment>
-<segment>
+<wire x1="39.37" y1="45.974" x2="45.72" y2="45.974" width="0.1524" layer="91"/>
+<label x="41.91" y="45.974" size="1.778" layer="95"/>
+</segment>
+<segment>
