File: src/USB_JST-XH_Converter.kicad_pcb (KiCad board)
At the start: 2 copper layers, 55.9 x 35.9 mm, 52 parts, among them SW1 SS-12D00G3, SW2 SML-E12V8WT86, U1 TCKE805NAWSON10B_TOS-REC, U2 TLP293

Commit message: シルク周りの微修正
Parts:
- added G***: LOGO, USB_JST-XH_Converter:メカテック部ロゴ拡大4, F.Cu at (172.0, 97.3)
